File: mmdvm_hs-hat.sch (KiCad schematic (older format))
At the start: 69 parts, among them P1 BOOT0, P2 DISPLAY, P3 SMA, P4 STLINK, SW1 SW_DIP_x01, U1 ADF7021, U2 STM32F103C8T6, X1 TCXO, Y1 8MHz

Commit message: The commit of MMDVM Hat VHF project
Parts:
- removed AE1: AN1603_433, MMDVM:AN1603, symbol Antenna_Dipole
- added L5: 20n, Resistors_SMD:R_0402, symbol L
- C1: value 6p8 -> 15p; MPN GJM1555C1H6R8BB01D -> GJM0225C1E150JB1L; SPN 81-GJM1555C1H6R8BB1D -> 81-GJM0225C1E150JB1L
- C12: value 470p -> 82p; MFR Murata Electronics -> TKD; MPN GRM155R71H471KA01D -> C0402CH1C820J02C; SPN 81-GRM36X471K50 -> 810-C0402CH1C820J02C
- C13: value 15n -> 2.7n; MFR Murata Electronics -> AVX; MPN GRM155R71C153KA01D -> 04025C272JAT2A; SPN 81-GRM155R71C153KA1D -> 581-04025C272JAT2A; SPR Mouser -> Taiyo Yuden
- C14: value 1n -> 200p; MPN GRM155R60J102KA01D -> 81-GCM1555C1H201FA6D; SPN 81-GRM155R60J102KA1D -> 81-GCM1555C1H201FA6D
- C27, C28: value 100n -> 15p; MPN GCM155R71C104JA55D -> GJM0225C1E150JB1L; SPN 81-GCM155R71C104JA5D -> 81-GJM0225C1E150JB1L
- C4: value 10p -> 18p; MPN GRM1555C1E100GA01D -> GRM1555C1H180JA1D; SPN 81-GRM1555C1E100GA1D -> 81-GRM1555C1H180JA1D
- C5: value 4p7 -> 12p; MPN GRM1555C1H4R7CA01D -> GRM1555C1H120FA1D; SPN 81-GRM1555C1H4R7CA1D -> 81-GRM1555C1H120FA1D
- C6: value 6p8 -> 10p
- L1: value 22n -> 150n; MFR Coilcraft -> TDK; MPN 0402AF-220XJLU -> MLG1005SR15JTD25; SPN 994-0402AF-220XJLU -> 810-MLG1005SR15JTD25
- L2: value 20n -> 130n; MFR TE Connectivity / Sigma Inductors -> TDK; MPN 36501E20NJTDG -> MLG1005SR13JTD25; SPN 279-36501E20NJTDG -> 810-MLG1005SR13JTD25
- L3: value 13n -> 100n; MPN 0402CS-13NXJLU -> 0402HPH-R10XJLW; SPN 994-0402CS-13NXJLU -> 994-0402HPH-R10XJLW
- L4: value 27n -> 200n; MPN 0402CS-27NXJLU -> 0402AF-201XJLU; SPN 994-0402CS-27NXJLU -> 994-0402AF-201XJLU
- R3: value 3k8 -> 3k6; MFR Susumu -> Panasonic; MPN RR0510P-3831-D -> ERA-2AEB362X; SPN 754-RR0510P-3831D -> 667-ERA-2AEB362X
- R4: value 3r9 -> 2r; MPN CRCW04023R90FKED -> CRCW04022R00FKED; SPN 71-CRCW04023R90FKED -> 71-CRCW0402-2-E3
- R5: value 560 -> 3.4K; MPN ERA-2AEB561X -> ERA-2AEB3401X; SPN 667-ERA-2AEB561X -> 667-ERA-2AEB3401X
- R6: value 270 -> 1.65K; MPN ERA-2AEB271X -> ERA-2AEB1651X; SPN 667-ERA-2AEB271X -> 667-ERA-2AEB1651X
Connections:
- net labels removed: RF
- wire segments 262 -> 267
- no-connect marks 28 -> 25
Other:
- moved on the sheet: C10, C11, C12, C13, C14, C15, C17, C18, C19, C2, C20, C22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
